File: Archivos Kicad/Termometro.kicad_pcb (KiCad board)
At the start: 2 copper layers, 53.3 x 67.8 mm, 22 parts, among them SW1 SW_Push, SW2 SW_Push, SW3 SW_Push, SW4 SW_Push, U1 LM358, U2 CC56-12EWA

Commit message: Minientrenador con deco BCD a 7 seg
Parts:
- removed D1: 1N4148, Diodes_ThroughHole:D_DO-35_SOD27_P7.62mm_Horizontal
- removed H3, H4: MountingHole, MountingHole:MountingHole_3.2mm_M3
- removed R1: 2k2, LibreriaCustumLemos:R_Axial_DIN0207_L6.3mm_D2.5mm_P10.16mm_Horizontal
- removed R2: 1k, LibreriaCustumLemos:R_Axial_DIN0207_L6.3mm_D2.5mm_P10.16mm_Horizontal
- removed R7: 4700, LibreriaCustumLemos:R_Axial_DIN0207_L6.3mm_D2.5mm_P10.16mm_Horizontal
- removed U1: LM358, Housings_DIP:DIP-8_W7.62mm_LongPads
- added H1: MountingHole, MountingHole:MountingHole_3.2mm_M3, F.Cu at (160.5, 126.6)
- added H2: MountingHole, MountingHole:MountingHole_3.2mm_M3, F.Cu at (118.9, 36.7)
- added U3: 74LS47, Package_DIP:DIP-16_W7.62mm_Socket, F.Cu at (132.9, 78.6)
- moved R6 38.5 mm to (116.9, 79.4), turned to 90 degrees
- moved U2 34.5 mm to (141.8, 48.9), turned to 90 degrees
- moved R3 27.8 mm to (127.5, 79.4), turned to 90 degrees
- moved R5 23.1 mm to (124.0, 79.4), turned to 90 degrees
- moved R4 14.9 mm to (120.4, 79.4)
- moved A1 9.27 mm to (158.3, 89.0)
- moved R10 9.11 mm to (133.6, 108.8)
- moved R11 9.11 mm to (123.5, 108.8)
- moved R12 9.11 mm to (130.2, 108.8)
- moved R8 9.11 mm to (126.8, 108.8)
- moved R9 9.11 mm to (120.1, 119.0)
- moved SW4 9.11 mm to (153.2, 127.1)
- moved SW3 9.11 mm to (123.4, 127.2)
- moved SW1 9.11 mm to (133.3, 127.1)
- moved SW2 9.11 mm to (143.3, 127.1)
Connections:
- A1 pad 10: /d -> /C
- A1 pad 11: /e -> /D
- A1 pad 12: /f -> /CC1
- A1 pad 13: /g -> /CC2
- A1 pad 14: /DPX -> /CC3
- A1 pad 15: /CC3 -> /CC4
- A1 pad 16: /CC4 -> unconnected-(A1-Pad16)
- A1 pad 20: Net-(A1-Pad20) -> unconnected-(A1-Pad20)
- A1 pad 5: /CC1 -> unconnected-(A1-Pad5)
- A1 pad 6: /CC2 -> unconnected-(A1-Pad6)
- A1 pad 7: /a -> /DPX
- A1 pad 8: /b -> /A
- A1 pad 9: /c -> /B
Routing:
- net /DPX: track 23.2 -> 82.5 mm, vias 0 -> 2
- net +5V: track 117.9 -> 175.3 mm
- net /a: track 66.8 -> 21.0 mm
- net GND: track 24.7 -> 56.9 mm
- net Net-(R3-Pad2): track 54.2 -> 22.5 mm, vias 0 -> 2
- net Net-(A1-Pad20): track 26.4 -> 0.00 mm
- net /g: track 31.4 -> 53.3 mm, vias 2 -> 0
- net /D: track 0.00 -> 21.7 mm, vias 0 -> 2
- net /d: track 10.2 -> 29.4 mm
- net Net-(R1-Pad1): track 18.7 -> 0.00 mm
- net /CC4: track 30.4 -> 12.1 mm
- net /c: track 11.9 -> 28.1 mm
- net /A: track 0.00 -> 15.7 mm
- net Net-(D1-Pad2): track 15.1 -> 0.00 mm
- net /B: track 0.00 -> 14.0 mm, vias 0 -> 2
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- removed copper zone on B.Cu, net GND
Other:
- board outline removed
- board text removed: "AED 3"
